File: KiCad/FloppyRider.kicad_pcb (KiCad board)
At the start: 2 copper layers, 88.9 x 59.7 mm, 29 parts, among them J1 PC disk controller interface, J2 IBM Diskette Host power, J3 IBM 51TD Diskette unit, J4 Alternative power connector, Q1 SS8050, SW1 Reset, SW2 Write prot, U1 74LS08, U2 74LS02, U3 74LS06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

Commit message: Version 2 board
Parts:
- added JP1: External override, Connector_PinHeader_2.54mm:PinHeader_1x02_P2.54mm_Vertical, F.Cu at (170.8, -74.9)
- added R14: 10K, Resistor_SMD:R_0603_1608Metric, F.Cu at (129.9, -52.8)
- added SW3: Write protection EXTERNAL, mis_partes:PinHeader_2x03_P2.54mm_Vertical CUSTOM, F.Cu at (155.6, -73.4)
- moved H2 152.4 mm to (188.7, -26.2)
- moved H3 152.4 mm to (188.7, -78.2)
- moved B1 152.4 mm to (141.7, -59.2)
- moved H1 152.4 mm to (107.4, -78.2)
- moved H4 152.4 mm to (107.4, -26.2)
- moved J1 152.4 mm to (184.9, -33.8)
- moved J2 152.4 mm to (116.3, -31.2)
- moved J3 152.4 mm to (125.2, -31.2)
- moved J4 152.4 mm to (136.7, -37.6)
- moved R1 152.4 mm to (177.3, -74.4)
- moved R10 152.4 mm to (177.3, -49.0)
- moved R11 152.4 mm to (177.3, -46.5)
- moved R13 152.4 mm to (177.3, -66.8)
- moved R2 152.4 mm to (177.3, -71.9)
- moved R3 152.4 mm to (177.3, -69.3)
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Connections:
- B1 pad 1: Net-(B1-Pad1) -> unconnected-(B1-Pad1)
- B1 pad 13: Net-(B1-Pad13) -> unconnected-(B1-Pad13)
- B1 pad 15: Net-(B1-Pad15) -> unconnected-(B1-Pad15)
- B1 pad 17: Net-(B1-Pad17) -> unconnected-(B1-Pad17)
- B1 pad 19: Net-(B1-Pad19) -> unconnected-(B1-Pad19)
- B1 pad 2: Net-(B1-Pad2) -> unconnected-(B1-Pad2)
- B1 pad 24: Net-(B1-Pad24) -> unconnected-(B1-Pad24)
- J1 pad 10: Net-(J1-Pad10) -> unconnected-(J1-Pad10)
- J1 pad 14: Net-(J1-Pad14) -> unconnected-(J1-Pad14)
- J1 pad 2: Net-(J1-Pad2) -> unconnected-(J1-Pad2)
- J1 pad 4: Net-(J1-Pad4) -> unconnected-(J1-Pad4)
- J1 pad 6: Net-(J1-Pad6) -> unconnected-(J1-Pad6)
- J2 pad 11: Net-(J2-Pad11) -> unconnected-(J2-Pad11)
- J2 pad 13: Net-(J2-Pad13) -> unconnected-(J2-Pad13)
- J2 pad 15: Net-(J2-Pad15) -> unconnected-(J2-Pad15)
- J2 pad 17: Net-(J2-Pad17) -> unconnected-(J2-Pad17)
- J2 pad 19: Net-(J2-Pad19) -> unconnected-(J2-Pad19)
- J2 pad 21: Net-(J2-Pad21) -> unconnected-(J2-Pad21)
- J2 pad 23: Net-(J2-Pad23) -> unconnected-(J2-Pad23)
- J2 pad 25: Net-(J2-Pad25) -> unconnected-(J2-Pad25)
- J2 pad 27: Net-(J2-Pad27) -> unconnected-(J2-Pad27)
- J2 pad 29: Net-(J2-Pad29) -> unconnected-(J2-Pad29)
- J2 pad 3: Net-(J2-Pad3) -> unconnected-(J2-Pad3)
- J2 pad 31: Net-(J2-Pad31) -> unconnected-(J2-Pad31)
- J2 pad 33: Net-(J2-Pad33) -> unconnected-(J2-Pad33)
- J2 pad 35: Net-(J2-Pad35) -> unconnected-(J2-Pad35)
- J2 pad 7: Net-(J2-Pad7) -> unconnected-(J2-Pad7)
- J2 pad 9: Net-(J2-Pad9) -> unconnected-(J2-Pad9)
- J3 pad 23: Net-(J3-Pad23) -> unconnected-(J3-Pad23)
- J3 pad 3: Net-(J3-Pad3) -> unconnected-(J3-Pad3)
- J3 pad 35: Net-(J3-Pad35) -> unconnected-(J3-Pad35)
- J4 pad 4: Net-(J4-Pad4) -> unconnected-(J4-Pad4)
- SW2 pad 1: Net-(SW2-Pad1) -> unconnected-(SW2-Pad1)
- SW2 pad 4: /write_protected -> Net-(JP1-Pad1)
- SW2 pad 6: Net-(SW2-Pad6) -> unconnected-(SW2-Pad6)
- U3 pad 12: Net-(U3-Pad12) -> unconnected-(U3-Pad12)
- U3 pad 13: Net-(U3-Pad13) -> unconnected-(U3-Pad13)
- U4 pad 10: Net-(U4-Pad10) -> unconnected-(U4-Pad10)
- U4 pad 11: Net-(U4-Pad11) -> unconnected-(U4-Pad11)
- U4 pad 12: Net-(U4-Pad12) -> unconnected-(U4-Pad12)
- U4 pad 13: Net-(U4-Pad13) -> unconnected-(U4-Pad13)
- U4 pad 8: Net-(U4-Pad8) -> unconnected-(U4-Pad8)
- U4 pad 9: Net-(U4-Pad9) -> unconnected-(U4-Pad9)
Routing:
- net Net-(JP1-Pad1): track 0.00 -> 29.6 mm
- net /write_erase_gate_prot: track 9.25 -> 34.2 mm
- net /index: track 61.8 -> 39.9 mm
- net /drive_b: track 89.8 -> 72.1 mm
- net /write_protected: track 17.4 -> 32.5 mm
- net /+24V: track 62.1 -> 49.1 mm
- net /8_write_erase_gate: track 61.1 -> 72.9 mm
- net /8_file_data: track 37.3 -> 47.9 mm
- net /direction: track 41.9 -> 52.0 mm
- net /8_index: track 33.1 -> 42.9 mm
- net /disk_chng_rdy_neg: track 18.7 -> 28.2 mm, vias 0 -> 1
- net /8_head_engage: track 74.3 -> 66.5 mm, vias 1 -> 2
- net /track_0_neg: track 15.2 -> 22.8 mm
- net GND: track 282.1 -> 289.2 mm, vias 0 -> 1
- net /write_erase_gate: track 28.5 -> 35.5 mm
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Other:
- net class 24v removed
- net class Default removed
- net class power removed
- board text added: "Install jumper JP1 if external write protection switch is not installed"
- board text added: "Leave internal write protection switch in ON position if external write protection switch is installed"
- board text added: "Write protection EXTERNAL"
- board text added: "write protection OFF"
- board text added: "write protection ON"
- board text removed: "write prot OFF"
- board text removed: "write prot ON"
